File: Hardware/SparkFun_RTK_Postcard.kicad_pcb (KiCad board)
At the start: 4 copper layers, 43.2 x 43.2 mm, 151 parts, among them J1 USB_C_Receptacle, J11 Val**, J2 SMA_Edge, J4 Qwiic_RA, J5 Val**, J6 U.FL, J7 Qwiic_RA, J8 JST_Locking_4, Q1 MBT3904DW1, SW4 Reset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

Commit message: Reduce paste on ESP32. Update to smaller schematic symbols.
Change to SparkFun library LG290P version.
Parts:
- J11: value Val** -> 1x10
- J5: value Val** -> 1x09
- JP7: value ~ -> SHLD
- turned F1 to 180 degrees
- turned R1 to 90 degrees
- turned R10 to 0 degrees
- turned R11 to 180 degrees
- turned R12 to 180 degrees
- turned R13 to 0 degrees
- turned R14 to 90 degrees
- turned R15 to 0 degrees
- turned R16 to 90 degrees
- turned R17 to -90 degrees
- turned R18 to -90 degrees
- turned R19 to 90 degrees
- turned R2 to 90 degrees
- turned R20 to 0 degrees
- turned R3 to 90 degrees
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Connections:
- F1 pad 1: Net-(F1-Pad1) -> VBUS
- F1 pad 2: VBUS -> Net-(F1-Pad2)
- J1 pad VBUS: Net-(F1-Pad1) -> Net-(F1-Pad2)
- JP6 pad 3: Net-(JP6-B) -> Net-(JP6-C)
- R1 pad 1: Net-(J1-CC2) -> GND
- R1 pad 2: GND -> Net-(J1-CC2)
- R10 pad 1: Net-(Q1B-B2) -> CH342-~{DTR}
- R10 pad 2: CH342-~{DTR} -> Net-(Q1B-B2)
- R11 pad 1: Net-(Q1A-B1) -> CH342-~{RTS}
- R11 pad 2: CH342-~{RTS} -> Net-(Q1A-B1)
- R12 pad 1: ESP35/DeviceSense -> GND
- R12 pad 2: GND -> ESP35/DeviceSense
- R13 pad 1: 3.3V -> ESP_~{RESET}
- R13 pad 2: ESP_~{RESET} -> 3.3V
- R14 pad 1: Net-(JP8-A) -> Net-(D6-A)
- R14 pad 2: Net-(D6-A) -> Net-(JP8-A)
- R15 pad 1: 3.3V -> ESP35/DeviceSense
- R15 pad 2: ESP35/DeviceSense -> 3.3V
- R16 pad 1: Net-(JP1-A) -> Net-(D9-A)
- R16 pad 2: Net-(D9-A) -> Net-(JP1-A)
- R17 pad 1: Net-(JP6-B) -> SDA_1
- R17 pad 2: SDA_1 -> Net-(JP6-C)
- R18 pad 1: Net-(JP6-A) -> SCL_1
- R18 pad 2: SCL_1 -> Net-(JP6-A)
- R19 pad 1: Net-(J2-In) -> Net-(D3-A2)
- R19 pad 2: Net-(D3-A2) -> Net-(J2-In)
- R2 pad 1: Net-(J1-CC1) -> GND
- R2 pad 2: GND -> Net-(J1-CC1)
- R20 pad 1: Net-(J6-In) -> Net-(D3-A2)
- R20 pad 2: Net-(D3-A2) -> Net-(J6-In)
- R3 pad 1: Net-(JP5-A) -> Net-(D2-A)
- R3 pad 2: Net-(D2-A) -> Net-(JP5-A)
- R4 pad 1: Net-(JP2-A) -> Net-(D1-A)
- R4 pad 2: Net-(D1-A) -> Net-(JP2-A)
- R5 pad 1: Net-(JP3-A) -> Net-(D4-A)
- R5 pad 2: Net-(D4-A) -> Net-(JP3-A)
- R6 pad 1: VCC_RF -> Net-(C3-Pad1)
- R6 pad 2: Net-(C3-Pad1) -> VCC_RF
- R7 pad 1: Net-(D5-PadC) -> V_BCKP
- R7 pad 2: V_BCKP -> Net-(D5-K)
- R8 pad 1: LG-RXD3 -> Net-(J8-Pin_3)
- R8 pad 2: Net-(J8-Pin_3) -> LG-RXD3
- R9 pad 1: 5V -> 3V3_EN
- R9 pad 2: 3V3_EN -> 5V
Routing:
- net Net-(F1-Pad2): track 0.00 -> 11.0 mm
- net Net-(F1-Pad1): track 11.0 -> 0.00 mm
- net Net-(JP6-C): track 0.00 -> 3.28 mm, vias 0 -> 1
- net Net-(JP6-B): track 3.28 -> 0.00 mm, vias 1 -> 0
- net Net-(D5-PadC): track 2.04 -> 0.00 mm
- net Net-(D5-K): track 0.00 -> 2.04 mm
