File: Hardware/SparkFun_RTK_Postcard.kicad_sch (KiCad schematic)
At the start: 76 parts, among them J1 USB_C_Receptacle, J10 Conn_01x06, J2 Conn_01x05, J3 JST_2mm_LiPo, J4 Qwiic_RA, J5 SMA_Edge, J7 Qwiic_RA, J8 JST_Locking_4, J9 I2C, Q1 MBT3904DW1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

Commit message: Rotate silkscreen. Add AIO pin.
Parts:
- removed J3: JST_2mm_LiPo, SparkFun-Connector:JST_SMD_2.0mm-2, symbol SparkFun-Connector:Conn_01x02_JST_2mm_LiPo
- removed J5: SMA_Edge, SparkFun-Connector:SMA_Edge, symbol SparkFun-RF:SMA_EdgeMount
- removed TP5: PTH, SparkFun-Connector:TestPoint-1.0mm, symbol SparkFun-Connector:TestPoint_1.0mm
- added C12: 1.0uF, SparkFun-Capacitor:C_0603_1608Metric, symbol SparkFun-Capacitor:1.0uF_0603_16V_10%
- added D7: PESD0603-240, SparkFun-Capacitor:C_0603_1608Metric, symbol SparkFun-DiscreteSemi:D_TVS_0603
- added D8: BAT60A, SparkFun-Semiconductor-Standard:SOD-323, symbol SparkFun-DiscreteSemi:D_Schottky_3A_10V_0.28V
- added J3: Conn_01x04, SparkFun-Connector:1x04, symbol SparkFun-Connector:Conn_01x04
- added J6: U.FL, SparkFun-Connector:U.FL, symbol SparkFun-RF:U.FL
Connections:
- net 3.3V: now also C12.1, D7.2 (A2)
- net 5V: now also D8.C; no longer F1.2
- net CH342-~{DTR}: now also U4.23 (~{DTR0}); no longer U4.15 (~{DTR1})
- net CH342-~{RTS}: now also U4.19 (~{RTS0}); no longer U4.11 (~{RTS1})
- net ESP1/TX: now also U4.20 (RXD0); no longer U4.12 (RXD1)
- net ESP3/RX: now also U4.21 (TXD0); no longer U4.13 (TXD1)
- net GND: now also C12.2, D7.1 (A1), J6.2 (Ext)
- net LG-RXD1: now also U4.13 (TXD1); no longer U4.21 (TXD0)
- net LG-RXD2: now also U5.34 (IO22)
- net LG-TXD1: now also U4.12 (RXD1); no longer U4.20 (RXD0)
- net LG-TXD2: now also U5.35 (IO21)
- net SCL: now also U5.26 (IO20)
- net SDA: now also U5.27 (IO7)
- net at C6.1, D3.2 (A2), L1.2: now also J6.1 (In)
- net ESP14/AIO: now reaches J10.1 (Pin_1)
- net ESP14/AIO: now also U5.18 (IOA14)
- net SHLD_SCK: now reaches U5.12 (IOA32)
- net SHLD_SCK: now also J3.1 (Pin_1)
- net SHLD_POCI: now reaches U5.15 (IOA25)
- net SHLD_POCI: now also J3.2 (Pin_2)
- net SHLD_PICO: now reaches U5.16 (IOA26)
- net SHLD_PICO: now also J3.3 (Pin_3)
- net SHLD_~{CS}: now reaches U5.17 (IOA27)
- net SHLD_~{CS}: now also J3.4 (Pin_4)
- net ESP12: no longer names the net of U5.19 (IOA12)
- net ESP15: no longer names the net of U5.21 (IOA15)
- net ESP2: no longer names the net of U5.22 (IOA2)
- net ESP5: no longer names the net of U5.29 (IO5)
- new net: D8.A, F1.2
- no-connect marks 14 -> 13
Other:
- note added: "Coplanar Waveguide Calculation: JLC04081H-7628 Stackup Copper Thickness (1oz): 1.4mil/0.035mm Board thickness: 0.8mm Dielectric thickness (layer 1 to 2): 0.2mm Er: 4.4 Polygon Isolation: 8mil/0.2032mm RF Trace Width: 13.48mil/0.3424mm https://jlcpcb.com/pcb-impedance-calculator"
- note added: "Prevent backfeed from external 5V"
- note removed: "Coplanar Waveguide Calculation: Copper Thickness (1oz): 1.4mil/0.035mm Board thickness: 1.6mm Dielectric thickness (layer 1 to 2): 0.2mm Er: 4.6 Polygon Isolation: 8mil/0.2032mm RF Trace Width: 13.74mil/0.349mm https://chemandy.com/calculators/coplanar-waveguide-with-ground-calculator.htm"
- moved on the sheet: C11, F1, J1, J10, J2, J8, J9, Q1A, Q1B, R1, R10, R11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

Commit message: Fix PPS. Add SMA. Change to 1.6mm. Add BT LED. Add I2C bus. Connect RST to LG290P..
Parts:
- removed C13: 0.1uF, SparkFun-Capacitor:C_0603_1608Metric, symbol SparkFun-Capacitor:0.1uF_0603_25V_20%
- removed J10: Conn_01x06, SparkFun-Connector:1x06, symbol SparkFun-Connector:Conn_01x06
- removed J2: Conn_01x05, SparkFun-Connector:1x05, symbol SparkFun-Connector:Conn_01x05
- removed J3: Conn_01x04, SparkFun-Connector:1x04, symbol SparkFun-Connector:Conn_01x04
- removed J9: I2C, SparkFun-Connector:1x04, symbol SparkFun-Connector:I2C_01x04
- added D9: Blue, SparkFun-LED:LED_0603_1608Metric_Blue, symbol SparkFun-LED:LED_Blue_0603
- added J11: 1x10, SparkFun-Connector:1x10, symbol SparkFun-Connector:Postcard_Mainboard_10
- added J2: SMA_Edge, SparkFun-Connector:SMA_Edge, symbol SparkFun-RF:SMA_EdgeMount
- added J5: 1x09, SparkFun-Connector:1x09, symbol SparkFun-Connector:Postcard_Mainboard_9
- added JP1: BT, SparkFun-Jumper:Jumper_2_NC_Trace, symbol SparkFun-Jumper:SolderJumper_2_Bridged
- added JP6: I²C-EXT, SparkFun-Jumper:Jumper_3_NC-2_Trace, symbol SparkFun-Jumper:SolderJumper_3_Bridged123
- added R16, R17, R18: 2.2k, SparkFun-Resistor:R_0603_1608Metric, symbol SparkFun-Resistor:2.2k_0603
- added R19, R20: 0, SparkFun-Resistor:R_0402_1005Metric, symbol SparkFun-Resistor:0_0402
- R9: value 10k -> 100k; symbol SparkFun-Resistor:10k_0603 -> SparkFun-Resistor:100k_0603; PROD_ID RES-00824 -> RES-07828
- U2: value AP2112K-3.3 -> RT9080-3.3; symbol SparkFun-Regulator:AP2112K-3.3 -> SparkFun-Regulator:RT9080-3.3; Iq 55µA -> 4µA; PROD_ID VREG-12457 -> VREG-19034
Connections:
- net PPS is gone; now on net LG-PPS: JP3.2 (B)
- net 3.3V: now also J11.9 (Pin_9), JP6.2 (C)
- net 3V3_EN: now also J11.2 (Pin_2)
- net 5V: now also J5.2; no longer C7.1, U4.7 (VDD5), U4.8 (VBUS)
- net ESP14/AIO: now also J11.6 (Pin_6)
- net GND: now also D9.1 (K), J11.10 (Pin_10), J2.2 (Ext), J5.1
- net LG-EVENT: now also J11.1 (Pin_1)
- net LG-PPS: now also U5.28 (IO8), J11.4 (Pin_4)
- net LG-RTK: now also J11.5 (Pin_5)
- net LG-RXD3: now also J5.4
- net LG-TXD3: now also J8.2 (Pin_2), J5.5; no longer J8.3 (Pin_3)
- net LG-~{RESET}: now also U5.13 (IOA33), J11.3 (Pin_3)
- net SHLD_PICO: now also J5.7
- net SHLD_POCI: now also J5.8
- net SHLD_SCK: now also J5.9
- net SHLD_~{CS}: now also J5.6
- net at R8.2: now also J8.3 (Pin_3); no longer J8.2 (Pin_2)
- net VBUS: now reaches D8.A, F1.2
- net VBUS: now also C7.1, U4.7 (VDD5), U4.8 (VBUS)
- net at C6.1, D3.2 (A2), L1.2: now also R19.2, R20.2; no longer J6.1 (In)
- net SDA_1: now reaches U5.20 (IOA13)
- net SDA_1: now also J4.3 (Pin_3), J7.3 (Pin_3), R17.2
- net BT_STATUS: now reaches U5.24 (IOA4)
- net BT_STATUS: now also JP1.2 (B)
- net SCL_1: now reaches U5.33 (IO19)
- net SCL_1: now also J4.4 (Pin_4), J7.4 (Pin_4), R18.2
- net SCL renamed SCL_0
- net SCL_0: now also J11.7 (Pin_7); no longer J4.4 (Pin_4), J7.4 (Pin_4)
- net SDA renamed SDA_0
- net SDA_0: now also J11.8 (Pin_8); no longer J4.3 (Pin_3), J7.3 (Pin_3)
- new net: J2.1 (In), R19.1
- new net: JP1.1 (A), R16.1
- new net: D9.2 (A), R16.2
- new net: JP6.3 (B), R17.1
- new net: J6.1 (In), R20.1
- new net: JP6.1 (A), R18.1
Other:
- note added: "Coplanar Waveguide Calculation: JLC04161H-7628 Stackup Copper Thickness (1oz): 1.4mil/0.035mm Board thickness: 1.6mm Dielectric thickness (layer 1 to 2): 0.2mm Er: 4.4 Polygon Isolation: 7mil/0.1778mm RF Trace Width: 11.1mil/0.2819mm https://jlcpcb.com/pcb-impedance-calculator"
- note added: "Internal I²C (0) is for display, GNSS config (future), fuel guage, etc. External I²C (1) is for (future) peripheral communication."
- note added: "No internal I²C0 pull-ups because LG290P has internal resistors."
- note added: "Prevent USB backfeed from external 5V"
- note added: "RADIO Port"
- note added: "The I²C ports are used as follows: I²C0 - Internal I²C I²C1 - External I²C"
- note added: "The ports are used as follows: UART1 - Configure in and NMEA output over USB UART2 - RTCM correction input and NMEA output over ESP32 Bluetooth UART3 - NMEA output to embedded system"
- note removed: "Coplanar Waveguide Calculation: JLC04081H-7628 Stackup Copper Thickness (1oz): 1.4mil/0.035mm Board thickness: 0.8mm Dielectric thickness (layer 1 to 2): 0.2mm Er: 4.4 Polygon Isolation: 8mil/0.2032mm RF Trace Width: 13.48mil/0.3424mm https://jlcpcb.com/pcb-impedance-calculator"
- note removed: "Generally speaking the ports are used as follows: UART1 - Configure in and NMEA output over USB UART2 - RTCM correction input and NMEA output over ESP32 Bluetooth UART3 - NMEA output to embedded system"
- note removed: "No external I²C pull-ups because LG290P has internal resistors."
- note removed: "Prevent backfeed from external 5V"
- moved on the sheet: C1, C2, C3, C4, C5, C6, C7, C8, D1, D2, D3, D4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

Commit message: Add panel files
Connections:
- net LG-EVENT: now also U5.28 (IO8)
- net LG-PPS: now also U5.4 (IA36); no longer U5.28 (IO8)
- net LG-RTK: now also U5.9 (IA34)
Other:
- note added: "No external I²C0 pull-ups because LG290P has internal resistors."
- note removed: "No internal I²C0 pull-ups because LG290P has internal resistors."
- title: LG290P Triband GNSS Receiver Breakout -> RTK Postcard (LG290P Quadband GNSS)
Changed lines of the file:
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@@
 	(paper "USLedger")
 	(title_block
-		(title "LG290P Triband GNSS Receiver Breakout")
+		(title "RTK Postcard (LG290P Quadband GNSS)")
 		(date "2024-08-21")
 		(rev "v10")
@@
 	(wire
 		(pts
+			(xy 339.09 100.33) (xy 337.82 100.33)
+		)
+		(stroke
+			(width 0)
+			(type default)
+		)
+	)
+	(wire
+		(pts
 			(xy 262.89 74.93) (xy 260.35 74.93)
 		)
@@
 	(wire
 		(pts
+			(xy 339.09 105.41) (xy 337.82 105.41)
+		)
+		(stroke
+			(width 0)
+			(type default)
+		)
+	)
+	(wire
+		(pts
 			(xy 90.17 154.94) (xy 90.17 161.29)
 		)
@@
 		)
 	)
-	(text "No internal I²C0 pull-ups because \nLG290P has internal resistors."
+	(text "No external I²C0 pull-ups because \nLG290P has internal resistors."
 		(exclude_from_sim no)
 		(at 385.064 76.962 0)
@@
 		)
 	)
+	(global_label "LG-PPS"
+		(shape input)
+		(at 339.09 105.41 0)
+		(fields_autoplaced yes)
+		(effects
+			(font
+				(size 1.27 1.27)
+			)
+			(justify left)
+		)
+		(property "Intersheetrefs" "${INTERSHEET_REFS}"
+			(at 349.6952 105.41 0)
+			(effects
+				(font
+					(size 1.27 1.27)
+				)
+				(justify left)
+				(hide yes)
+			)
+		)
+	)
 	(global_label "ESP35{slash}DeviceSense"
 		(shape input)
@@
 		)
 	)
+	(global_label "LG-EVENT"
+		(shape input)
+		(at 339.09 69.85 0)
+		(fields_autoplaced yes)
+		(effects
+			(font
+				(size 1.27 1.27)
+			)
+			(justify left)
+		)
+		(property "Intersheetrefs" "${INTERSHEET_REFS}"
+			(at 351.6304 69.85 0)
+			(effects
+				(font
+					(size 1.27 1.27)
+				)
+				(justify left)
+				(hide yes)
+			)
+		)
+	)
 	(global_label "ESP0{slash}~{BOOT}"
 		(shape input)
@@
 		)
 	)
-	(global_label "LG-PPS"
+	(global_label "SDA_0"
 		(shape input)
-		(at 339.09 69.85 0)
+		(at 82.55 242.57 0)
 		(fields_autoplaced yes)
 		(effects
@@
 		)
 		(property "Intersheetrefs" "${INTERSHEET_REFS}"
-			(at 349.6952 69.85 0)
+			(at 91.2804 242.57 0)
 			(effects
 				(font
@@
 		)
 	)
-	(global_label "SDA_0"
+	(global_label "LG-PPS"
 		(shape input)
-		(at 82.55 242.57 0)
+		(at 149.86 158.75 90)
 		(fields_autoplaced yes)
 		(effects
@@
 		)
 		(property "Intersheetrefs" "${INTERSHEET_REFS}"
-			(at 91.2804 242.57 0)
+			(at 149.86 148.1448 90)
 			(effects
 				(font
@@
 		)
 	)
-	(global_label "LG-PPS"
+	(global_label "LG-RTK"
 		(shape input)
-		(at 149.86 158.75 90)
+		(at 339.09 100.33 0)
 		(fields_autoplaced yes)
 		(effects
@@
 		)
 		(property "Intersheetrefs" "${INTERSHEET_REFS}"
-			(at 149.86 148.1448 90)
+			(at 349.4533 100.33 0)
 			(effects
 				(font

Commit message: Add housing 3D file
Parts:
- JP7: value ~ -> SHLD
Changed lines of the file:
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@@
 			)
 		)
-		(property "Value" "~"
+		(property "Value" "SHLD"
 			(at 19.05 87.63 90)
 			(effects

Commit message: Reduce paste on ESP32. Update to smaller schematic symbols.
Change to SparkFun library LG290P version.
Parts:
- U2: IMax (none) -> 600mA; VMax 6V -> 5.5V
- U3: symbol LG209P:LG290P -> SparkFun-GPS:LG290P
Connections:
- net 3.3V: now also D5.2 (A), R13.2, R15.2; no longer D5.A, R13.1, R15.1
- net 3V3_EN: now also R9.1; no longer R9.2
- net 5V: now also D8.1 (K), R9.2; no longer D8.C, R9.1
- net CH342-~{DTR}: now also R10.1; no longer R10.2
- net CH342-~{RTS}: now also R11.1; no longer R11.2
- net ESP35/DeviceSense: now also R12.2, R15.1; no longer R12.1, R15.2
- net ESP_~{RESET}: now also R13.1; no longer R13.2
- net GND: now also R1.1, R12.1, R2.1; no longer R1.2, R12.2, R2.2
- net LG-RXD3: now also R8.2; no longer R8.1
- net SCL_1: now also R18.1; no longer R18.2
- net SDA_1: now also R17.1; no longer R17.2
- net VBUS: now also D8.2 (A), F1.1; no longer D8.A, F1.2
- net VCC_RF: now also R6.2; no longer R6.1
- net V_BCKP: now also R7.1; no longer R7.2
- net at R19.1: now also C6.1, D3.2 (A2), L1.2, R20.1; no longer J2.1 (In)
- net at J8.3 (Pin_3): now also R8.1; no longer R8.2
- net at R16.1: now also D9.2 (A); no longer JP1.1 (A)
- net at R16.2: now also JP1.1 (A); no longer D9.2 (A)
- net at JP5.1 (A): now also R3.2; no longer R3.1
- net at Q1.5 (B2): now also R10.2; no longer R10.1
- net at J1.VBUS: now also F1.2; no longer F1.1
- net at D2.2 (A): now also R3.1; no longer R3.2
- net at JP6.3 (C): now also R17.2; no longer R17.1
- net at J6.1 (In): now also R20.2; no longer R20.1
- net at JP8.1 (A): now also R14.2; no longer R14.1
- net at J1.B5 (CC2): now also R1.2; no longer R1.1
- net at C3.1, C4.1, L1.1: now also R6.1; no longer R6.2
- net at D1.2 (A): now also R4.1; no longer R4.2
- net at JP2.1 (A): now also R4.2; no longer R4.1
- net at R5.1: now also D4.2 (A); no longer JP3.1 (A)
- net at R5.2: now also JP3.1 (A); no longer D4.2 (A)
- net at D6.2 (A): now also R14.1; no longer R14.2
- net at JP6.1 (A): now also R18.2; no longer R18.1
- net at J1.A5 (CC1): now also R2.2; no longer R2.1
- net at Q1.2 (B1): now also R11.2; no longer R11.1
- new net: J2.1 (In), R19.2
- new net: D5.1 (K), R7.2
Other:
- moved on the sheet: D1, D2, D4, D6, D9
