File: Hardware/SparkFun_RTK_Postcard.kicad_sch (KiCad schematic)
At the start: 84 parts, among them J1 USB_C_Receptacle, J11 1x10, J2 SMA_Edge, J4 Qwiic_RA, J5 1x09, J6 U.FL, J7 Qwiic_RA, J8 JST_Locking_4, Q1 MBT3904DW1, SW4 Reset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

Commit message: Update sch/pcb with smaller sch parts. Update prod panel with 10% paste reduction.
Parts:
- U2: IMax (none) -> 600mA; VMax 6V -> 5.5V
- U3: symbol LG209P:LG290P -> SparkFun-GPS:LG290P
Connections:
- net 3.3V: now also D5.2 (A), R13.2, R15.2; no longer D5.A, R13.1, R15.1
- net 3V3_EN: now also R9.1; no longer R9.2
- net 5V: now also D8.1 (K), R9.2; no longer D8.C, R9.1
- net CH342-~{DTR}: now also R10.1; no longer R10.2
- net CH342-~{RTS}: now also R11.1; no longer R11.2
- net ESP35/DeviceSense: now also R12.2, R15.1; no longer R12.1, R15.2
- net ESP_~{RESET}: now also R13.1; no longer R13.2
- net GND: now also R1.1, R12.1, R2.1; no longer R1.2, R12.2, R2.2
- net LG-RXD3: now also R8.2; no longer R8.1
- net SCL_1: now also R18.1; no longer R18.2
- net SDA_1: now also R17.1; no longer R17.2
- net VBUS: now also D8.2 (A), F1.1; no longer D8.A, F1.2
- net VCC_RF: now also R6.2; no longer R6.1
- net V_BCKP: now also R7.1; no longer R7.2
- net at R19.1: now also C6.1, D3.2 (A2), L1.2, R20.1; no longer J2.1 (In)
- net at J8.3 (Pin_3): now also R8.1; no longer R8.2
- net at R16.1: now also D9.2 (A); no longer JP1.1 (A)
- net at R16.2: now also JP1.1 (A); no longer D9.2 (A)
- net at JP5.1 (A): now also R3.2; no longer R3.1
- net at Q1.5 (B2): now also R10.2; no longer R10.1
- net at J1.VBUS: now also F1.2; no longer F1.1
- net at D2.2 (A): now also R3.1; no longer R3.2
- net at JP6.3 (C): now also R17.2; no longer R17.1
- net at J6.1 (In): now also R20.2; no longer R20.1
- net at JP8.1 (A): now also R14.2; no longer R14.1
- net at J1.B5 (CC2): now also R1.2; no longer R1.1
- net at C3.1, C4.1, L1.1: now also R6.1; no longer R6.2
- net at D1.2 (A): now also R4.1; no longer R4.2
- net at JP2.1 (A): now also R4.2; no longer R4.1
- net at R5.1: now also D4.2 (A); no longer JP3.1 (A)
- net at R5.2: now also JP3.1 (A); no longer D4.2 (A)
- net at D6.2 (A): now also R14.1; no longer R14.2
- net at JP6.1 (A): now also R18.2; no longer R18.1
- net at J1.A5 (CC1): now also R2.2; no longer R2.1
- net at Q1.2 (B1): now also R11.2; no longer R11.1
- new net: J2.1 (In), R19.2
- new net: D5.1 (K), R7.2
Other:
- moved on the sheet: D1, D2, D4, D6, D9

Commit message: Update to v9 and current libraries.
Parts:
- removed Q1: MBT3904DW1, SparkFun-Semiconductor-Standard:SOT-323, symbol SparkFun-DiscreteSemi:Q_NPN_DUAL
- added Q2: MBT3904DW1, SparkFun-Semiconductor-Standard:SOT-363_SC-70-6, symbol SparkFun-DiscreteSemi:Q_NPN_DUAL
- BT1: value 6.8mm_ML414H -> ML414H
- C2: PROD_ID CAP-11015 -> CAP-25001
- D3: symbol SparkFun-DiscreteSemi:D_TVS_0402 -> SparkFun-DiscreteSemi:D_TVS_0402_14V; Rating (none) -> 14VWM/40VC
- D7: symbol SparkFun-DiscreteSemi:D_TVS_0603 -> SparkFun-DiscreteSemi:D_TVS_0603_24V; Rating (none) -> 24VWM/45VC
- G5: footprint SparkFun-Aesthetic:SparkFun_Logo_8mm -> (none)
- J11: footprint SparkFun-Connector:1x10 -> SparkFun-Connector:1x10_P2.54mm
- J2: footprint SparkFun-Connector:SMA_Edge -> SparkFun-Connector:SMA_Edge_8mm; symbol SparkFun-RF:SMA_EdgeMount -> SparkFun-RF:SMA_EdgeMount_8mm; PROD_ID CONN-08289 -> CONN-19593
- J4, J7: footprint SparkFun-Connector:JST_SMD_1.0mm-4_RA -> SparkFun-Connector:JST_1x04_P1.0mm_Horizontal_SMD; symbol SparkFun-Connector:Qwiic_Right_Angle -> SparkFun-Connector:Qwiic_Horizontal
- J5: footprint SparkFun-Connector:1x09 -> SparkFun-Connector:1x09_P2.54mm
- J8: footprint SparkFun-Connector:JST_SMD_1.25mm-4_Locking -> SparkFun-Connector:JST_1x04_P1.25mm_Locking_Horizontal_SMD; symbol SparkFun-Connector:Conn_01x04_JST_1.25mm_Locking -> SparkFun-Connector:Conn_01x04_JST_P1.25mm_Locking_Horizontal_SMD
- JP1: value BT -> ~
- JP2: value PWR -> ~
- JP3: value PPS -> ~
- JP4: value VSEL -> ~
- JP5: value RTK -> ~
- JP6: value I²C-EXT -> ~
- JP7: value SHLD -> ~
- JP8: value STAT -> ~
- SW4: value Reset -> SMD_4.6x2.8mm_h2.5mm
- SW5: value Boot -> SMD_4.6x2.8mm_h2.5mm
- TP1, TP2, TP3, TP4, TP6: value PTH -> 1.0mm
- U1: symbol SparkFun-DiscreteSemi:D_TVS_ESD_USB -> SparkFun-DiscreteSemi:D_TVS_ESD_USB_5V; Rating (none) -> 5VWM/9VC
- U2: Imax 600mA -> (none)
- U3: footprint LG290P:Quectel_LG290P -> SparkFun-GNSS:Quectel_LG290P; symbol SparkFun-GPS:LG290P -> SparkFun-GNSS:LG290P
Connections:
- net CH342-~{DTR}: now also Q2.6 (C1)
- net CH342-~{RTS}: now also Q2.4 (E2)
- net ESP0/~{BOOT}: now also Q2.1 (E1)
- net ESP_~{RESET}: now also Q2.3 (C2)
- net at R10.2: now also Q2.5 (B2)
- net at R11.2: now also Q2.2 (B1)
Other:
- moved on the sheet: C3, C4, C6, D3, D8, J2, J6, L1, R1, R19, R2, R20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

Commit message: Add MFi. Update symbols. Use main library sym/fps.
Parts:
- removed Q2: MBT3904DW1, SparkFun-Semiconductor-Standard:SOT-363_SC-70-6, symbol SparkFun-DiscreteSemi:Q_NPN_DUAL
- removed R19, R20: 0, SparkFun-Resistor:R_0402_1005Metric, symbol SparkFun-Resistor:0_0402
- added C14: 0.1uF, SparkFun-Capacitor:C_0603_1608Metric, symbol SparkFun-Capacitor:0.1uF_0603_25V_20%
- added JP10: ~, SparkFun-Jumper:Jumper_2_NO, symbol SparkFun-Jumper:SolderJumper_2_Open
- added JP9: ~, SparkFun-Jumper:Jumper_2_NC_Trace, symbol SparkFun-Jumper:SolderJumper_2_Bridged
- added Q1: MBT3904DW1, SparkFun-Semiconductor-Standard:SOT-363_SC-70-6, symbol SparkFun-DiscreteSemi:Q_NPN_DUAL
- added U6: MFI343S00177, SparkFun-Semiconductor-Standard:DFN-8_3x2mm_P0.5mm_EP1.66x1.5mm, symbol SparkFun-IC-Special-Function:MFI343S00177
- JP4: value ~ -> VCC
- JP6: value ~ -> I2C
- SW4: value SMD_4.6x2.8mm_h2.5mm -> RESET
- SW5: value SMD_4.6x2.8mm_h2.5mm -> BOOT
Connections:
- net 3.3V: now also C14.1, U6.8 (VCC)
- net CH342-~{DTR}: now also Q1.1 (E1)
- net CH342-~{RTS}: now also Q1.4 (E2)
- net ESP0/~{BOOT}: now also Q1.6 (C1)
- net ESP_~{RESET}: now also Q1.3 (C2)
- net GND: now also C14.2, U6.1 (GND), U6.4 (GND), U6.7 (GND)
- net SCL_0: now also U6.6 (SCL)
- net SDA_0: now also U6.5 (SDA)
- net at C6.1, D3.2 (A2), L1.2: now also JP10.2 (B), JP9.2 (B)
- net at J2.1 (In): now also JP9.1 (A)
- net at R11.2: now also Q1.2 (B1)
- net at R10.2: now also Q1.5 (B2)
- net at J6.1 (In): now also JP10.1 (A)
Other:
- note added: "Fix the FP discrepancy on the ESP boot transistor"
- note added: "MFi Authentication Coprocessor"
- moved on the sheet: C1, C2, C5, C8, D7, D8, R10, R11, R12, R13, R15, R9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
